File: Digit/Digit.kicad_sch (KiCad schematic)
At the start: 48 parts, among them J1 4s Batt, J10 Linear Actuator, J11 UV Bulb, J12 Sparkmax Pwr, J14 Sparkmax PWM, J16 AS7341, J17 FAERIE Lasers, J18 SHT30, J2 12V, J3 VIC CAN, J4 Debug, J5 EF Motor, J6 Cam 1 Pwr Conn, J7 Lynx Servos, J8 EF Laser, J9 CAM 2 Pwr Conn, Q1 SSM3K329R_LF, Q2 SSM3K329R_LF, U1 TJA1051T/3, U2 BD622xF

Commit message: URC '25 - V2
Parts:
- removed A1: Adafruit Feather ESP32 V2, Module:Adafruit_Feather, symbol adafruit_feather_esp32_v2:Adafruit_Feather_ESP32_V2
- removed C1: 4.7 nF, Capacitor_SMD:C_0603_1608Metric_Pad1.08x0.95mm_HandSolder, symbol Device:C
- removed J10: Linear Actuator, Connector_Molex:Molex_Mini-Fit_Jr_5566-02A_2x01_P4.20mm_Vertical, symbol Connector:Conn_01x02_Socket
- removed J11: UV Bulb, Connector_Molex:Molex_Mini-Fit_Jr_5566-02A_2x01_P4.20mm_Vertical, symbol Connector:Conn_01x02_Pin
- removed J14: Sparkmax PWM, Connector_Molex:Molex_Mini-Fit_Jr_5566-02A_2x01_P4.20mm_Vertical, symbol Connector:Conn_01x02_Pin
- removed J17: FAERIE Lasers, Connector_Molex:Molex_Mini-Fit_Jr_5566-02A_2x01_P4.20mm_Vertical, symbol Connector:Conn_01x02_Pin
- removed J18: SHT30, Connector_Molex:Molex_Mini-Fit_Jr_5566-04A_2x02_P4.20mm_Vertical, symbol Connector:Conn_01x04_Pin
- removed J4: Debug, Connector_PinHeader_2.54mm:PinHeader_2x03_P2.54mm_Vertical, symbol Connector:Conn_01x06_Socket
- removed J5: EF Motor, Connector_Molex:Molex_Mini-Fit_Jr_5566-02A_2x01_P4.20mm_Vertical, symbol Connector:Conn_01x02_Socket
- removed J8: EF Laser, Connector_Molex:Molex_Mini-Fit_Jr_5566-02A_2x01_P4.20mm_Vertical, symbol Connector:Conn_01x02_Socket
- removed JP1: CAN Term Jmp, Jumper:SolderJumper-3_P1.3mm_Open_Pad1.0x1.5mm, symbol Jumper:SolderJumper_3_Open
- removed Q1: SSM3K329R_LF, Digit:SOT-23F_TOS, symbol SSM3K329R_LF:SSM3K329R_LF
- removed Q2: SSM3K329R_LF, Digit:SOT-23F_TOS, symbol Nmos:SSM3K329R_LF
- removed R1: 10Ω, Resistor_SMD:R_0603_1608Metric_Pad0.98x0.95mm_HandSolder, symbol Device:R_US
- removed R14: 330, Resistor_SMD:R_0603_1608Metric_Pad0.98x0.95mm_HandSolder, symbol Device:R_US
- removed R15: 0, Resistor_SMD:R_0603_1608Metric_Pad0.98x0.95mm_HandSolder, symbol Device:R_US
- added C1: 4.7 nF, Capacitor_SMD:C_0603_1608Metric_Pad1.08x0.95mm_HandSolder, symbol Device:C_Small
- added C10, C11: 1uF, Capacitor_SMD:C_0603_1608Metric_Pad1.08x0.95mm_HandSolder, symbol Device:C_Small
- added C12: 100u, Capacitor_SMD:C_0603_1608Metric_Pad1.08x0.95mm_HandSolder, symbol Device:C
- added C13: 10u, Capacitor_SMD:C_0603_1608Metric_Pad1.08x0.95mm_HandSolder, symbol Device:C
- added C6, C7: 100pF, Capacitor_SMD:C_0603_1608Metric_Pad1.08x0.95mm_HandSolder, symbol Device:C_Small
- added C8: 10uF, Capacitor_SMD:C_0603_1608Metric_Pad1.08x0.95mm_HandSolder, symbol Device:C_Small
- added C9: 0.1 uF, Capacitor_SMD:C_0603_1608Metric_Pad1.08x0.95mm_HandSolder, symbol Device:C
- added D5: 15, Diode_SMD:D_SOD-123, symbol Device:D_Zener
- added D6, D7: D_TVS_Dual_ACA, SHC:SG-WLL-3-1, symbol Device:D_TVS_Dual_ACA
- added D8: Inolux_IN-PI554FCH, LED_SMD:LED_Inolux_IN-PI554FCH_PLCC4_5.0x5.0mm_P3.2mm, symbol LED:Inolux_IN-PI554FCH
- added D9: TVS, SHC:SOD-323HEUS2H_TOS, symbol Device:D_Zener
- added J13: EF Motor, Lin ac, Laser, Connector_Molex:Molex_Mini-Fit_Jr_5566-06A_2x03_P4.20mm_Vertical, symbol Connector_Generic:Conn_02x03_Top_Bottom
- added J15: UV Bulb, Sparkmax PWM, Lasers, Connector_Molex:Molex_Mini-Fit_Jr_5566-06A_2x03_P4.20mm_Vertical, symbol Connector_Generic:Conn_02x03_Top_Bottom
- added Q2: SSM3K329R_LF, Digit:SOT-23F_TOS, symbol SSM3K329R_LF:SSM3K329R_LF
- added Q3: PMOS, Package_TO_SOT_SMD:TO-252-2, symbol Simulation_SPICE:PMOS
- added Q4: SSM3K329R_LF, Digit:SOT-23F_TOS, symbol Nmos:SSM3K329R_LF
- added R1, R14: 10k, Resistor_SMD:R_0603_1608Metric_Pad0.98x0.95mm_HandSolder, symbol Device:R_Small_US
- added R16: 10, Resistor_SMD:R_0603_1608Metric_Pad0.98x0.95mm_HandSolder, symbol Device:R_Small_US
- added R17: 50k, Resistor_SMD:R_0603_1608Metric_Pad0.98x0.95mm_HandSolder, symbol Device:R_US
- added R18: 330, Resistor_SMD:R_0603_1608Metric_Pad0.98x0.95mm_HandSolder, symbol Device:R_US
- added R19: 0Ω, Resistor_SMD:R_0603_1608Metric_Pad0.98x0.95mm_HandSolder, symbol Device:R_Small_US
- added U3: ESP32 DOIT Devkit V1, esp32_devkit_v1_doit:esp32_devkit_v1_doit, symbol ESP 32 DOIT devkit V1:ESP32_DOIT_devkit_V1
- C2: value C -> 100u; footprint (none) -> Capacitor_SMD:C_0603_1608Metric_Pad1.08x0.95mm_HandSolder
- C3: value 0.1 μF -> 100 nF
- C4: value 1 μF -> 47 nF
- C5: value C -> 10u; footprint (none) -> Capacitor_SMD:C_0603_1608Metric_Pad1.08x0.95mm_HandSolder
- D1: value VBATT -> BATT
- D4: value 24V -> TVS; footprint (none) -> SHC:SOD-323HEUS2H_TOS
- J16: value AS7341 -> AS7341 or SHT30
- R11, R12: value 60Ω -> 60
- R2, R3, R5, R7: value 10 kΩ -> 10k
- R6: value 3.8 kΩ -> 3.32k
- R8: value 3.1 kΩ -> 2.21k
Connections:
- net +12V: now also C2.1, C5.1, D4.1 (K), J7.3 (Pin_3), U2.6 (VREF), C8.1, D5.1 (K), J13.6 (Pin_6), J15.4 (Pin_4), Q3.3 (S); no longer J2.2 (Pin_2), J7.1 (Pin_1)
- net +3.3V: now also U3.16 (3.3V)
- net +5V: now also C3.1, C9.1, D8.3 (VDD), J15.6 (Pin_6), U3.15 (VIN)
- net +BATT: now also C12.1, C13.1, D9.1 (K); no longer C2.1, C5.1, D4.1 (K)
- net 12V_ADC: now also D6.3 (A2), U3.2 (GPI36/A0)
- net 5V_ADC: now also D7.1 (A1), U3.5 (GPI35/A7)
- net BATT_ADC: now also D6.1 (A1), U3.3 (GPI39/A3)
- net CAN_H: now also C7.2
- net CAN_L: now also C6.1
- net CAN_RX: now also U3.10 (GPIO27/A17)
- net CAN_TX: now also U3.11 (GPIO14/A16)
- net GND: now also J7.1 (Pin_1), C1.1, C10.2, C11.2, C12.2, C13.2, C6.2, C7.1, C8.2, C9.2, D6.2 (common), D7.2 (common), D8.1 (VSS), D9.2 (A), J15.2 (Pin_2), Q2.2, Q4.2, R1.1, R14.1, R17.2, R18.2, U3.14 (GND), U3.17 (GND); no longer C3.1, J7.3 (Pin_3)
- net I2C_SCL: now also U3.29 (GPIO22/SCL)
- net I2C_SDA: now also U3.26 (GPIO21/SDA)
- net LINAC_FIN: now also R1.2, U3.24 (GPIO18/SCK)
- net LINAC_NEG: now also C10.1, J13.2 (Pin_2)
- net LINAC_POS: now also C11.1, J13.5 (Pin_5)
- net LINAC_RIN: now also R14.2, U3.25 (GPIO19/MISO)
- net MOTOR_FLT: now also U3.20 (GPIO4/A10)
- net MOTOR_IN1: now also U3.7 (GPIO33/A5)
- net MOTOR_IN2: now also U3.8 (GPIO25/A18)
- net MOTOR_OUT1: now also J13.4 (Pin_4)
- net MOTOR_OUT2: now also J13.1 (Pin_1)
- net UART_MISO: now also U3.21 (GPIO16/RX2)
- net UART_MOSI: now also U3.22 (GPIO17/TX2)
- net at R12.1: now also R11.2, C1.2
- new net: Q4.3, R16.2
- new net: Q2.3, R19.2
- new net: J15.1 (Pin_1), R18.1
- new net: J15.3 (Pin_3), R19.1
- new net: D5.2 (A), Q3.2 (G), R17.1
- new net: J13.3 (Pin_3), R16.1
- new net 12V_IN: J2.2 (Pin_2), Q3.1 (D)
- new net LASER_NMOS: Q2.1, Q4.1, U3.30 (GPIO23/MOSI)
- new net NEO_LED_DIN: D8.2 (DIN), U3.13 (GPIO13/A14)
- new net SPARK_PWM: J15.5 (Pin_5), U3.9 (GPIO26/A19)
- no-connect marks 16 -> 17
Other:
- note added: "12V (5.8V) 20mA"
- note added: "12V >6.5A"
- note added: "12V Protection Circuit"
- note added: "14.8V ~11A"
- note added: "3.3V >2mA"
- note added: "Extra pin!!!!!!"
- note added: "Neopixel Debug LED"
- note added: "PWM"
- note added: "rip too small D: Never not checking size again I didn't even know they made stuff that small"
- note removed: "(Vdrop 5.8V) 12V 20mA"
- note removed: "12V ~6.5A"
- note removed: "14.8V"
- note removed: "3.3V ?mA"
- moved on the sheet: A3, A4, C2, C3, C4, C5, D1, D2, D3, D4, J1, J12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
