File: Arm/Arm.kicad_pcb (KiCad board)
At the start: 2 copper layers, 97 x 107 mm, 56 parts, among them J10 SparkMAX XT60 F, J11 CAN OUT, J12 Axis 0, J13 SparkMAX XT60 F, J14 Encoder 0, J2 Encoder Bundle, J3 CAN IN, J4 5V Swtich Power, J5 Power IN XT60 M, J6 SparkMAX XT60 F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

Commit message: URC '25 - V2
Parts:
- removed A1, A2: Adafruit_Feather_HUZZAH32_ESP32, Module:Adafruit_Feather
- added C7: 0.1 uF, Capacitor_SMD:C_0603_1608Metric_Pad1.08x0.95mm_HandSolder, F.Cu at (86.3, 87.1)
- added D5: Inolux_IN-PI554FCH, LED_SMD:LED_Inolux_IN-PI554FCH_PLCC4_5.0x5.0mm_P3.2mm, F.Cu at (80.9, 87.2)
- added R16: 10K ohm, Resistor_SMD:R_0603_1608Metric_Pad0.98x0.95mm_HandSolder, F.Cu at (64.8, 64.2)
- added U8: ~, ESP 32 DOIT devkit V1:esp32_devkit_v1_doit, F.Cu at (87.1, 74.4)
- J12: value Axis 0 -> SparkMAX XT60 F; footprint Connector_Molex:Molex_Mini-Fit_Jr_5566-04A_2x02_P4.20mm_Vertical -> Connector_AMASS:AMASS_XT60-F_1x02_P7.20mm_Vertical
- J8: footprint Connector_Molex:Molex_Mini-Fit_Jr_5566-04A_2x02_P4.20mm_Vertical -> Connector_AMASS:AMASS_XT30U-F_1x02_P5.0mm_Vertical
- R1: moved to F.Cu
- R5: value 3.8K Ohm -> 3.32K Ohm
- R7: value 3.1K Ohm -> 2.21K ohm
- U6: footprint Arm:Pololu 3730 -> ESP 32 DOIT devkit V1:esp32_devkit_v1_doit
- moved J3 62.7 mm to (49.3, 106.4)
- moved J6 55.5 mm to (85.0, 128.0), turned to 90 degrees
- moved J11 46.4 mm to (49.3, 114.6)
- moved G*** 44.6 mm to (130.6, 99.3), turned to 90 degrees
- moved J8 43.0 mm to (113.3, 100.4), turned to -90 degrees
- moved J10 41.2 mm to (95.2, 128.0), turned to 90 degrees
- moved M1 39.2 mm to (132.5, 81.2)
- moved J4 35.0 mm to (79.5, 100.2), turned to 0 degrees
- moved J12 34.4 mm to (74.8, 128.0), turned to 90 degrees
- moved J13 27.0 mm to (105.5, 128.0), turned to 90 degrees
- moved U6 24.7 mm to (55.1, 74.4), turned to 180 degrees
- moved R1 23.9 mm to (64.7, 66.8), turned to 0 degrees
- moved R11 23.6 mm to (89.5, 89.9), turned to -90 degrees
- moved D4 23.4 mm to (89.5, 85.8), turned to -90 degrees
- moved R2 22.6 mm to (64.7, 66.8), turned to 180 degrees
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Connections:
- J12 pad 1: /Stepper A+ -> GND
- J12 pad 2: /Stepper A- -> +BATT
- J14 pad 2: /MOSI_ESP0 -> GND
- J14 pad 3: /MISO_ESP0 -> /CS_Encoder_0
- J14 pad 4: /CS_Encoder_0 -> /MOSI_ESP0
- J14 pad 5: GND -> /MISO_ESP0
- J8 pad 1: /ESP_RX-LYNX_TX -> +12V
- J8 pad 2: /ESP_TX-LYNX_RX -> GND
- R3 pad 1: +3.3V -> /3.3V_ADC
- U4 pad 1: /ESP0_RX-CAN_TX -> /ESP0_TX-CAN_TX
- U4 pad 4: /ESP0_TX-CAN_RX -> /ESP0_RX-CAN_RX
- U5 pad 1: /ESP1_RX-CAN_TX -> /ESP1_TX-CAN_TX
- U5 pad 4: /ESP1_TX-CAN_RX -> /ESP1_RX-CAN_RX
- U6 pad 10: +3.3V -> unconnected-(U6-GPIO27/A17-Pad10)
- U6 pad 11: unconnected-(U6-RESET-Pad11) -> /ESP0_RX-CAN_RX
- U6 pad 13: unconnected-(U6-BIN1-Pad13) -> /ESP0_TX-CAN_TX
- U6 pad 14: unconnected-(U6-BIN2-Pad14) -> GND
- U6 pad 15: unconnected-(U6-STALL/BEMFV-Pad15) -> +5V
- U6 pad 16: unconnected-(U6-BEMF-Pad16) -> /ESP0 3.3V
- U6 pad 17: /Stepper B- -> GND
- U6 pad 18: /Stepper B+ -> unconnected-(U6-GPIO15/A13-Pad18)
- U6 pad 19: /Stepper A- -> unconnected-(U6-GPIO2/A12-Pad19)
- U6 pad 2: +3.3V -> /12V_ADC
- U6 pad 20: /Stepper A+ -> unconnected-(U6-GPIO4/A10-Pad20)
- U6 pad 21: GND -> /ESP0_ESP1_SERIAL
- U6 pad 22: GND -> /ESP1_ESP0_SERIAL
- U6 pad 23: +BATT -> unconnected-(U6-GPIO05/CS-Pad23)
- U6 pad 24: +BATT -> /CLK_ESP0
- U6 pad 3: GND -> /BATT_ADC
- U6 pad 4: unconnected-(U6-STEP/AIN1-Pad4) -> /5V_ADC
- U6 pad 5: unconnected-(U6-DIR/AIN2-Pad5) -> /3.3V_ADC
- U6 pad 6: /MOSI_ESP0 -> /CS_Encoder_0
- U6 pad 7: /MISO_ESP0 -> /CS_Encoder_1
- U6 pad 8: /CLK_ESP0 -> /CS_Encoder_2
- U6 pad 9: /Axis 0 CS -> /CS_Encoder_3
Routing:
- net +12V: track 231.8 -> 135.5 mm
- net /ESP_TX-LYNX_RX: track 59.0 -> 0.00 mm
- net /ESP_RX-LYNX_TX: track 57.4 -> 0.00 mm
- net /Axis 0 CS: track 56.4 -> 0.00 mm, vias 2 -> 0
- net /Stepper B+: track 54.6 -> 0.00 mm
- net /Stepper B-: track 52.2 -> 0.00 mm
- net /Vehicle Control CAN+: track 104.6 -> 53.5 mm, vias 2 -> 0
- net +3.3V: track 172.7 -> 123.2 mm
- net /Stepper A-: track 45.9 -> 0.00 mm
- net /Stepper A+: track 45.3 -> 0.00 mm
- net /LED Debug: track 0.00 -> 43.1 mm, vias 0 -> 3
- net /Vehicle Control CAN-: track 96.3 -> 55.5 mm, vias 2 -> 0
- net +5V: track 295.0 -> 264.1 mm, vias 6 -> 3
- net /MOSI_ESP0: track 81.2 -> 53.0 mm, vias 0 -> 1
- net /CS_Encoder_1: track 92.5 -> 66.2 mm
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- added copper zone on F.Cu, net +5V
- added copper zone on B.Cu, net +BATT
Other:
- board text added: "ARM SOCKET V2 4/4/25 Brennan Begley"
- board text added: "AXIS 0 ENCODER MOSI 3.3V MISO GND CLK CS"
- board text added: "Fan +12V GND"
- board text removed: "ARM SOCKET V1 11/7/24 Brennan Begley"
- board text removed: "AXIS 0 ENCODER CS 3.3V GND MOSI CLK MISO"
- board text removed: "AXIS 0 MOTOR B+ A+ B- A-"
- board text removed: "RX TX"

Commit message: PCB Layout....
Parts:
- removed C2: 4.7 nf, Capacitor_SMD:C_0603_1608Metric_Pad1.08x0.95mm_HandSolder
- removed G*** (x3): LOGO, LOGO
- removed R12, R13: 60Ω, Resistor_SMD:R_0603_1608Metric_Pad0.98x0.95mm_HandSolder
- removed U6, U8: ~, ESP 32 DOIT devkit V1:esp32_devkit_v1_doit
- removed U7: RASPBERRY_PI_4B_4GB, Raspi:MODULE_RASPBERRY_PI_4B_4GB
- added C10: 0.1 uF, Capacitor_SMD:C_0603_1608Metric_Pad1.08x0.95mm_HandSolder, F.Cu at (128.2, 141.9)
- added C11: 4.7 nF, Capacitor_SMD:C_0603_1608Metric_Pad1.08x0.95mm_HandSolder, F.Cu at (128.2, 144.5)
- added C8: 0.1 uF, Capacitor_SMD:C_0603_1608Metric_Pad1.08x0.95mm_HandSolder, F.Cu at (123.8, 154.5)
- added C9: 0.1 uF, Capacitor_SMD:C_0603_1608Metric_Pad1.08x0.95mm_HandSolder, F.Cu at (128.2, 139.4)
- added R17: 60Ω, Resistor_SMD:R_0603_1608Metric_Pad0.98x0.95mm_HandSolder, F.Cu at (136.8, 116.7)
- added R18: 60Ω, Resistor_SMD:R_0603_1608Metric_Pad0.98x0.95mm_HandSolder, F.Cu at (136.8, 119.2)
- added U9: MCP251863T-E-9PX, Package_DFN_QFN:VQFN-28-1EP_5x5mm_P0.5mm_EP3.25x3.25mm, B.Cu at (63.2, 119.5)
- added Y3: 40Mhz Crystal, Crystal:Crystal_SMD_3225-4Pin_3.2x2.5mm, B.Cu at (69.6, 115.2)
- C1, C3, C5, R14, R15, R2, R3, R5, R7: moved to F.Cu
- C4: value 1 uF -> 13 pF; moved to F.Cu
- C6: value 0.1 uF -> 13 pF; moved to F.Cu
- U5: value TJA1051T -> ESP32-S3-DevKitC; footprint Package_SO:SOIC-8_3.9x4.9mm_P1.27mm -> Astra Lib:ESP32-S3-DevKitC; moved to F.Cu
- moved H2 169.0 mm to (185.2, 37.2), turned to -90 degrees
- moved H3 143.9 mm to (180.2, 37.2), turned to -90 degrees
- moved J5 138.1 mm to (20.8, 38.5), turned to 0 degrees
- moved J7 117.4 mm to (20.8, 59.0), turned to 0 degrees
- moved C5 114.1 mm to (123.8, 147.0), turned to 0 degrees
- moved C4 111.5 mm to (123.8, 144.5), turned to 0 degrees
- moved R3 108.3 mm to (128.2, 152.0), turned to 0 degrees
- moved R2 104.2 mm to (128.2, 149.5), turned to 0 degrees
- moved R4 104.1 mm to (128.2, 154.5)
- moved C6 103.6 mm to (123.8, 149.5)
- moved R1 102.2 mm to (128.2, 147.0)
- moved J6 102.0 mm to (20.8, 48.8), turned to 0 degrees
- moved H4 101.6 mm to (175.2, 37.2), turned to -90 degrees
- moved R7 100.9 mm to (132.5, 144.5), turned to 0 degrees
- moved R6 99.0 mm to (132.5, 141.9)
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Connections:
- C4 pad 1: +5V -> GND
- C4 pad 2: GND -> Net-(U9-OSC1)
- C6 pad 2: /ESP1 3.3V -> Net-(U9-OSC2)
- U5 pad 1: /ESP1_TX-CAN_TX -> /ESP0 3.3V
- U5 pad 2: GND -> /ESP0 3.3V
- U5 pad 4: /ESP1_RX-CAN_RX -> unconnected-(U5-GPIO4/ADC1_CH3-Pad4)
- U5 pad 5: /ESP1 3.3V -> unconnected-(U5-GPIO5/ADC1_CH4-Pad5)
- U5 pad 6: /Arm Motor CAN- -> unconnected-(U5-GPIO6/ADC1_CH5-Pad6)
- U5 pad 7: /Arm Motor CAN+ -> /ESP0_RX-CAN_RX
Routing:
- net +5V: track 264.1 -> 0.00 mm, vias 3 -> 0
- net +12V: track 135.5 -> 0.00 mm, vias 5 -> 0
- net +3.3V: track 123.2 -> 0.00 mm, vias 2 -> 0
- net +BATT: track 105.7 -> 0.00 mm, vias 5 -> 0
- net /CS_Encoder_3: track 83.7 -> 0.00 mm
- net /CLK_ESP0: track 76.4 -> 0.00 mm, vias 2 -> 0
- net /CS_Encoder_2: track 74.7 -> 0.00 mm, vias 2 -> 0
- net /MISO_ESP0: track 68.4 -> 0.00 mm
- net /CS_Encoder_1: track 66.2 -> 0.00 mm
- net /Vehicle Control CAN-: track 55.5 -> 0.00 mm
- net /Arm Motor CAN+: track 55.3 -> 0.00 mm
- net /Vehicle Control CAN+: track 53.5 -> 0.00 mm
- net /MOSI_ESP0: track 53.0 -> 0.00 mm, vias 1 -> 0
- net /CS_Encoder_0: track 51.4 -> 0.00 mm, vias 2 -> 0
- net /Arm Motor CAN-: track 45.2 -> 0.00 mm
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- removed copper zone on F.Cu, net +5V
- removed copper zone on B.Cu, net +BATT
- removed copper zone on F.Cu, net +BATT
Other:
- board size 97 x 107 mm -> 307 x 216.8 mm
- board text removed: "12V"
- board text removed: "12V GND"
- board text removed: "132mm x 107mm MAX SIZE"
- board text removed: "3.3V"
- board text removed: "3.3V CS1 CS2 CS3"
- board text removed: "5V"
- board text removed: "ARM SOCKET V2 4/4/25 Brennan Begley"
- board text removed: "AXIS 0 ENCODER MOSI 3.3V MISO GND CLK CS"
- board text removed: "BAT"
- board text removed: "BAT IN"
- board text removed: "BAT OUT"
- board text removed: "CAN TERMINATION"
- board text removed: "Fan +12V GND"
- board text removed: "H L"
- board text removed: "MAIN ESP"
- board text removed: "MOSI MISO CLK GND"
- board text removed: "MOTOR"
- board text removed: "MOTOR ESP"
- board text removed: "SWITCH PWR 5V GND"
- board text removed: "Spark Max"
- board text removed: "VIC CAN"

Commit message: Progrss on socket -FeedBack Fixes -PCB Layout and signal routing
Parts:
- removed C7: 0.1 uF, Capacitor_SMD:C_0603_1608Metric_Pad1.08x0.95mm_HandSolder
- removed D5: Inolux_IN-PI554FCH, LED_SMD:LED_Inolux_IN-PI554FCH_PLCC4_5.0x5.0mm_P3.2mm
- removed R1, R2, R3: 10K Ohm, Resistor_SMD:R_0603_1608Metric_Pad0.98x0.95mm_HandSolder
- removed R16, R4, R6: 10K ohm, Resistor_SMD:R_0603_1608Metric_Pad0.98x0.95mm_HandSolder
- removed R5: 3.32K Ohm, Resistor_SMD:R_0603_1608Metric_Pad0.98x0.95mm_HandSolder
- removed R7: 2.21K ohm, Resistor_SMD:R_0603_1608Metric_Pad0.98x0.95mm_HandSolder
- added R12: R_Small_US, Resistor_SMD:R_0603_1608Metric_Pad0.98x0.95mm_HandSolder, F.Cu at (93.0, 165.3)
- added R13: R_Small_US, Resistor_SMD:R_0603_1608Metric_Pad0.98x0.95mm_HandSolder, F.Cu at (92.9, 162.7)
- added R19: 2k ohm, Resistor_SMD:R_0603_1608Metric_Pad0.98x0.95mm_HandSolder, F.Cu at (92.9, 159.5)
- added R20: R_Small_US, Resistor_SMD:R_0603_1608Metric_Pad0.98x0.95mm_HandSolder, F.Cu at (93.2, 168.1)
- added R21: 10K ohm, Resistor_SMD:R_0603_1608Metric_Pad0.98x0.95mm_HandSolder, F.Cu at (92.2, 83.0)
- added R22: 10K ohm, Resistor_SMD:R_0603_1608Metric_Pad0.98x0.95mm_HandSolder, F.Cu at (98.2, 101.0)
- added R23: 10K ohm, Resistor_SMD:R_0603_1608Metric_Pad0.98x0.95mm_HandSolder, F.Cu at (96.1, 127.2)
- added R24: 10K ohm, Resistor_SMD:R_0603_1608Metric_Pad0.98x0.95mm_HandSolder, F.Cu at (144.7, 94.2)
- C4, C5, C6, R18: moved to B.Cu
- J12, J6, J7: footprint Connector_AMASS:AMASS_XT60-F_1x02_P7.20mm_Vertical -> Connector_AMASS:AMASS_XT60PW-F_1x02_P7.20mm_Horizontal
- J5: footprint Connector_AMASS:AMASS_XT60-M_1x02_P7.20mm_Vertical -> Connector_AMASS:AMASS_XT60PW-M_1x02_P7.20mm_Horizontal
- J8: value Lynx -> Digit 12V
- R10, R11: value 3.8K Ohm -> 10k ohm
- R8: value 3.8K Ohm -> 2.21K ohm
- R9: value 3.8K Ohm -> 3.32K ohm
- U9: footprint Package_DFN_QFN:VQFN-28-1EP_5x5mm_P0.5mm_EP3.25x3.25mm -> Package_SO:SSOP-28_5.3x10.2mm_P0.65mm
- moved H1 150.6 mm to (122.0, 171.5)
- moved H2 150.6 mm to (117.0, 171.5)
- moved H3 150.6 mm to (112.0, 171.5)
- moved H4 150.6 mm to (107.0, 171.5)
- moved D4 81.7 mm to (88.6, 168.8)
- moved D3 81.4 mm to (88.6, 165.8)
- moved D2 81.0 mm to (88.6, 162.7)
- moved D1 80.7 mm to (88.4, 159.5)
- moved JP1 78.6 mm to (101.8, 160.7)
- moved J11 74.3 mm to (85.2, 146.5), turned to 90 degrees
- moved J3 72.1 mm to (76.8, 146.5), turned to 90 degrees
- moved J10 66.0 mm to (55.1, 125.7)
- moved J9 63.9 mm to (100.6, 151.0)
- moved R15 62.3 mm to (106.7, 166.2)
- moved C10 62.3 mm to (159.8, 88.3)
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Connections:
- R10 pad 1: Net-(D3-A) -> /3.3V_ADC
- R11 pad 1: Net-(D4-A) -> /5V_ADC
- R8 pad 1: Net-(D1-A) -> /BATT_ADC
- R9 pad 1: Net-(D2-A) -> /12V_ADC
- U5 pad 10: unconnected-(U5-GPIO17/ADC2_CH6-Pad10) -> /ESP0_TX-CAN_TX
- U5 pad 11: /ESP0_TX-CAN_TX -> unconnected-(U5-GPIO18/ADC2_CH7-Pad11)
- U5 pad 21: unconnected-(U5-5V-Pad21) -> +5V
- U5 pad 27: /LED Debug -> unconnected-(U5-GPIO21-Pad27)
- U5 pad 28: /MISO_ESP0 -> /CS_Encoder_2
- U5 pad 3: +5V -> unconnected-(U5-CHIP_PU-Pad3)
- U5 pad 30: /CS_Encoder_2 -> /MISO_ESP0
- U5 pad 32: /MOSI_ESP0 -> /CS_Motor_CAN
- U5 pad 33: /CS_Motor_CAN -> /MOSI_ESP0
Routing:
- net /MISO_ESP0: track 0.00 -> 113.4 mm
- net /MOSI_ESP0: track 0.00 -> 107.3 mm
- net +5V: track 0.00 -> 97.0 mm, vias 0 -> 3
- net /CS_Encoder_2: track 0.00 -> 90.2 mm
- net /CS_Encoder_1: track 0.00 -> 64.6 mm
- net /CS_Encoder_3: track 0.00 -> 63.6 mm
- net +BATT: track 0.00 -> 60.4 mm
- net /Vehicle Control CAN-: track 0.00 -> 58.4 mm
- net /CLK_ESP0: track 0.00 -> 57.9 mm
- net +3.3V: track 0.00 -> 57.4 mm, vias 0 -> 2
- net /CS_Encoder_0: track 0.00 -> 53.3 mm
- net /Vehicle Control CAN+: track 0.00 -> 51.3 mm
- net /ESP0 3.3V: track 0.00 -> 48.9 mm, vias 0 -> 1
- net /Arm Motor CAN-: track 0.00 -> 30.1 mm
- net /Arm Motor CAN+: track 0.00 -> 29.7 mm
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- added copper zone on F.Cu, net +12V
- added copper zone on B.Cu, net +BATT
- added copper zone on F.Cu, net +BATT
Other:
- board size 307 x 216.8 mm -> 104.5 x 139.5 mm

Commit message: More Work on PCB
Moved some stuff around
Parts:
- added D1: LED, LED_SMD:LED_0603_1608Metric_Pad1.05x0.95mm_HandSolder, F.Cu at (235.6, 105.2)
- added D5: LED, LED_SMD:LED_0603_1608Metric_Pad1.05x0.95mm_HandSolder, F.Cu at (235.6, 107.8)
- added D6: LED, LED_SMD:LED_0603_1608Metric_Pad1.05x0.95mm_HandSolder, F.Cu at (235.6, 110.4)
- added D7: LED, LED_SMD:LED_0603_1608Metric_Pad1.05x0.95mm_HandSolder, F.Cu at (235.6, 113.0)
- C1, C11, R11, R14, R15, R17, R22, R24, R9: moved to B.Cu
- J10: footprint Connector_AMASS:AMASS_XT60-F_1x02_P7.20mm_Vertical -> Connector_AMASS:AMASS_XT60-M_1x02_P7.20mm_Vertical
- J11, J3: footprint Connector_AMASS:AMASS_XT30U-M_1x02_P5.0mm_Vertical -> Connector_AMASS:AMASS_XT30U-F_1x02_P5.0mm_Vertical
- J8: footprint Connector_AMASS:AMASS_XT30U-F_1x02_P5.0mm_Vertical -> Connector_AMASS:AMASS_XT30PW-F_1x02_P2.50mm_Horizontal
- moved C11 60.4 mm to (114.2, 130.4), turned to 90 degrees
- moved R17 57.7 mm to (116.2, 127.8), turned to 180 degrees
- moved C8 39.5 mm to (126.8, 128.0)
- moved C10 38.0 mm to (140.6, 121.0)
- moved C9 38.0 mm to (136.3, 136.1)
- moved R11 37.4 mm to (127.8, 90.0), turned to 180 degrees
- moved R21 36.3 mm to (127.8, 90.0)
- moved R18 31.8 mm to (112.2, 127.8)
- moved R9 20.9 mm to (104.8, 118.0), turned to 180 degrees
- moved R24 18.2 mm to (127.8, 87.5)
- moved R22 15.7 mm to (111.4, 109.5), turned to 180 degrees
- moved R10 13.7 mm to (111.4, 109.5)
- moved R23 12.6 mm to (104.8, 118.0)
- moved R8 9.24 mm to (127.8, 87.5), turned to 180 degrees
- moved C1 8.25 mm to (98.4, 163.2)
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Connections:
- R12 pad 1: Net-(D3-A) -> Net-(D6-K)
- R13 pad 1: Net-(D2-A) -> Net-(D1-K)
- R19 pad 1: Net-(D1-A) -> Net-(D5-K)
- R20 pad 1: Net-(D4-A) -> Net-(D7-K)
- U5 pad 16: unconnected-(U5-GPIO10/ADC1_CH9-Pad16) -> /12V_ADC
- U5 pad 31: /12V_ADC -> unconnected-(U5-GPIO0-Pad31)
Routing:
- net +3.3V: track 57.4 -> 91.4 mm
- net +5V: track 97.0 -> 119.1 mm, vias 3 -> 5
- net /ESP0 3.3V: track 48.9 -> 68.7 mm, vias 1 -> 2
- net /12V_ADC: track 0.00 -> 5.30 mm
- net /3.3V_ADC: track 0.00 -> 5.10 mm
- net /BATT_ADC: track 0.00 -> 5.00 mm
- net /5V_ADC: track 0.00 -> 4.97 mm
- net /Arm Motor CAN+: track 29.7 -> 34.5 mm
- net Net-(JP1-C): track 0.00 -> 2.54 mm
- net Net-(JP1-A): track 0.00 -> 2.41 mm
- net Net-(JP1-B): track 0.00 -> 2.34 mm
- net GND: track 0.00 -> 0.03 mm, vias 9 -> 11
- added copper zone on B.Cu, net Net-(C11-Pad2)

Commit message: So Close...
Parts:
- removed the D1 at (235.6, 105.2)
- removed the D1 at (88.4, 159.5)
- removed D2, D3, D4: LED, LED_SMD:LED_0603_1608Metric_Pad1.05x0.95mm_HandSolder
- added D1: LED, LED_SMD:LED_0603_1608Metric_Pad1.05x0.95mm_HandSolder, F.Cu at (87.1, 155.5)
- J8: footprint Connector_AMASS:AMASS_XT30PW-F_1x02_P2.50mm_Horizontal -> Connector_AMASS:AMASS_XT30U-F_1x02_P5.0mm_Vertical
- R23: moved to B.Cu
- R9: moved to F.Cu
- moved D5 165.8 mm to (75.9, 152.2), turned to 180 degrees
- moved D7 165.3 mm to (75.9, 155.5), turned to 180 degrees
- moved D6 154.5 mm to (86.9, 152.2), turned to 180 degrees
- moved J3 98.5 mm to (118.5, 57.2), turned to 0 degrees
- moved J11 87.3 mm to (118.5, 65.8), turned to 0 degrees
- moved R15 31.9 mm to (126.5, 142.2), turned to 90 degrees
- moved C1 29.4 mm to (124.0, 148.9), turned to 90 degrees
- moved C9 24.9 mm to (120.2, 117.0), turned to -90 degrees
- moved JP1 24.9 mm to (121.4, 145.5), turned to 90 degrees
- moved R14 24.5 mm to (121.2, 142.2), turned to -90 degrees
- moved C10 20.8 mm to (121.0, 127.9), turned to -90 degrees
- moved J9 18.8 mm to (83.0, 144.5), turned to 90 degrees
- moved R20 17.9 mm to (80.5, 155.5)
- moved R19 14.5 mm to (80.4, 152.2)
- moved R12 13.1 mm to (92.2, 152.2)
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Routing:
- net /CLK_ESP0: track 57.9 -> 134.3 mm
- net +12V: track 13.3 -> 83.8 mm, vias 0 -> 1
- net /Vehicle Control CAN-: track 58.4 -> 8.50 mm
- net +3.3V: track 91.4 -> 135.6 mm, vias 2 -> 3
- net /Vehicle Control CAN+: track 51.3 -> 8.50 mm
- net +5V: track 119.1 -> 159.2 mm, vias 5 -> 7
- net +BATT: track 60.4 -> 84.8 mm
- net /Arm Motor CAN-: track 30.1 -> 53.8 mm
- net /Arm Motor CAN+: track 34.5 -> 48.7 mm
- net /CS_Encoder_1: track 64.6 -> 72.5 mm
- net GND: track 0.03 -> 3.89 mm, vias 11 -> 17
- net /MOSI_ESP0: track 107.3 -> 110.3 mm
- net /3.3V_ADC: track 5.10 -> 2.55 mm
- net /MISO_ESP0: track 113.4 -> 112.4 mm
- net /ESP0_TX-CAN_TX: track 8.70 -> 7.82 mm
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
Commit message: The Unholy PCB
Parts:
- moved JP1 95.8 mm to (74.9, 61.8)
- moved C1 95.8 mm to (77.5, 65.1)
- moved R14 95.5 mm to (74.0, 59.2), turned to 0 degrees
- moved R15 94.5 mm to (81.2, 59.2), turned to 0 degrees
- moved J10 65.6 mm to (53.3, 60.1)
- moved J13 64.6 mm to (53.2, 72.8)
- moved J11 60.0 mm to (63.5, 41.8)
- moved J3 60.0 mm to (63.5, 33.2)
- moved J12 30.4 mm to (62.6, 138.2)
- moved J6 30.4 mm to (62.8, 120.2)
- moved J7 30.4 mm to (62.8, 84.7)
- moved J5 30.3 mm to (62.8, 109.5)
- moved J4 27.4 mm to (121.5, 146.2)
- moved J14 11.5 mm to (120.9, 65.1)
- moved J2 11.5 mm to (99.3, 65.9)
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Routing:
- net +BATT: track 84.8 -> 222.3 mm, vias 0 -> 4
- net /Arm Motor CAN-: track 53.8 -> 22.3 mm
- net /Arm Motor CAN+: track 48.7 -> 19.6 mm
- net +3.3V: track 135.6 -> 163.7 mm, vias 3 -> 5
- net /CLK_ESP0: track 134.3 -> 121.6 mm
- net /CS_Encoder_1: track 72.5 -> 61.0 mm
- net /MOSI_ESP0: track 110.3 -> 99.0 mm
- net /CS_Encoder_2: track 90.2 -> 80.7 mm
- net /MISO_ESP0: track 112.4 -> 105.1 mm
- net /CS_Encoder_0: track 54.1 -> 47.7 mm
- net /CS_Encoder_3: track 63.6 -> 60.4 mm
- net /3.3V_ADC: track 2.55 -> 4.30 mm
- net +5V: track 159.2 -> 159.8 mm
- net GND: track 3.89 -> 3.86 mm, vias 17 -> 808
- removed copper zone on B.Cu, net +BATT
- removed copper zone on F.Cu, net +BATT
Other:
- board size 104.5 x 139.5 mm -> 91.1 x 109 mm

Commit message: Had the plague
Parts:
- added kibuzzard-69541E91: G***, kibuzzard-69541E91, F.Cu at (90.2, 144.5)
- added kibuzzard-69541EDE: G***, kibuzzard-69541EDE, F.Cu at (90.2, 139.2)
- added kibuzzard-69541FE4: G***, kibuzzard-69541FE4, F.Cu at (82.0, 115.8)
- added kibuzzard-69542020: G***, kibuzzard-69542020, F.Cu at (82.0, 118.2)
- added kibuzzard-69542020: G***, kibuzzard-69542020, F.Cu at (82.0, 120.8)
- added kibuzzard-6954203E: G***, kibuzzard-6954203E, F.Cu at (82.8, 123.5)
- moved J11 23.9 mm to (69.0, 65.0)
- moved J3 23.9 mm to (69.0, 56.5)
- moved C5 13.7 mm to (113.0, 101.9), turned to -90 degrees
- moved Y3 12.7 mm to (127.0, 121.0), turned to 0 degrees
- moved C6 12.2 mm to (126.8, 118.1)
- moved C3 10.6 mm to (113.0, 113.8)
- moved C4 10.1 mm to (126.4, 123.9), turned to 180 degrees
- moved R14 8.16 mm to (78.2, 66.2), turned to 90 degrees
- moved JP1 6.81 mm to (80.7, 65.3), turned to 180 degrees
- moved C1 6.39 mm to (83.0, 61.9), turned to -90 degrees
- moved C8 4.53 mm to (122.2, 128.5)
- moved U9 4.53 mm to (117.5, 122.0)
- moved C10 4.53 mm to (116.5, 128.4)
- moved C9 3.85 mm to (116.8, 115.4), turned to 90 degrees
- moved C11 3.11 mm to (116.0, 135.5)
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Routing:
- net +5V: track 159.8 -> 117.0 mm, vias 7 -> 4
- net /Arm Motor CAN-: track 22.3 -> 11.5 mm
- net Net-(U9-OSC2): track 16.6 -> 6.60 mm
- net Net-(U9-OSC1): track 16.5 -> 7.12 mm
- net /ESP0_TX-CAN_TX: track 7.82 -> 14.0 mm
- net /CS_Motor_CAN: track 19.2 -> 25.0 mm
- net /MOSI_ESP0: track 99.0 -> 104.6 mm
- net /ESP0_RX-CAN_RX: track 16.1 -> 21.6 mm
- net /MISO_ESP0: track 105.1 -> 110.4 mm
- net /CLK_ESP0: track 121.6 -> 125.8 mm
- net Net-(D6-K): track 0.00 -> 3.59 mm
- net /Arm Motor CAN+: track 19.6 -> 16.8 mm
- net Net-(D5-K): track 0.00 -> 2.75 mm
- net Net-(U9-TXCAN): track 7.79 -> 5.89 mm
- net /ESP0 3.3V: track 69.4 -> 70.0 mm, vias 2 -> 3
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
Commit message: 1 PCB 2 PCB 3 PCB ...
Parts:
- moved R11 16.4 mm to (111.5, 92.5), turned to 0 degrees
- moved R21 16.4 mm to (111.5, 92.5), turned to 180 degrees
- moved C5 0.64 mm to (113.0, 101.2)
Connections:
- U5 pad 11: unconnected-(U5-GPIO18/ADC2_CH7-Pad11) -> /ESP0_RX-CAN_RX
- U5 pad 28: /CS_Encoder_2 -> unconnected-(U5-GPIO47-Pad28)
- U5 pad 4: unconnected-(U5-GPIO4/ADC1_CH3-Pad4) -> /CS_Encoder_2
- U5 pad 40: /5V_ADC -> unconnected-(U5-GPIO2/ADC1_CH1-Pad40)
- U5 pad 6: unconnected-(U5-GPIO6/ADC1_CH5-Pad6) -> /5V_ADC
- U5 pad 7: /ESP0_RX-CAN_RX -> unconnected-(U5-GPIO7/ADC1_CH6-Pad7)
Routing:
- net +BATT: track 222.3 -> 332.4 mm, vias 4 -> 2
- net +5V: track 117.0 -> 173.9 mm
- net /CS_Encoder_2: track 80.7 -> 28.7 mm
- net /ESP0_RX-CAN_RX: track 21.6 -> 6.75 mm
- net /Vehicle Control CAN+: track 8.83 -> 21.0 mm, vias 0 -> 1
- net /Vehicle Control CAN-: track 8.50 -> 15.8 mm, vias 0 -> 1
- net +3.3V: track 163.7 -> 163.0 mm, vias 5 -> 3
