File: Arm/Arm.kicad_pcb (KiCad board)
At the start: 2 copper layers, 92.4 x 109 mm, 91 parts, among them J10 SparkMAX XT60 F, J11 CAN OUT, J12 SparkMAX XT60 F, J13 SparkMAX XT60 F, J14 Encoder 0, J2 Encoder Bundle, J3 CAN IN, J4 5V Swtich Power, J5 Power IN XT60 M, J6 SparkMAX XT60 F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

Commit message: 2/3 Final Changes
Parts:
- removed kibuzzard-698ABA0B: G***, kibuzzard-698ABA0B
- added kibuzzard-69B0C619: G***, kibuzzard-69B0C619, B.Cu at (128.0, 152.0)
- J10, J13: footprint Connector_AMASS:AMASS_XT60PW-F_1x02_P7.20mm_Horizontal -> Connector_AMASS:AMASS_XT60-F_1x02_P7.20mm_Vertical
- moved kibuzzard-696EEFE3 89.4 mm to (55.2, 149.3), turned to 180 degrees
- moved J3 87.7 mm to (51.0, 140.1), turned to -90 degrees
- moved R15 81.6 mm to (53.2, 134.8), turned to 180 degrees
- moved J11 77.1 mm to (59.5, 140.1), turned to -90 degrees
- moved C1 75.4 mm to (56.1, 130.1), turned to 0 degrees
- moved J13 73.9 mm to (69.1, 64.4)
- moved R14 72.3 mm to (60.5, 134.8), turned to 180 degrees
- moved JP1 72.0 mm to (59.6, 132.3), turned to -90 degrees
- moved J10 42.2 mm to (81.1, 64.3)
- moved J6 11.4 mm to (62.8, 108.8)
- moved J12 6.13 mm to (62.8, 90.7)
- moved J7 6.13 mm to (58.1, 78.9)
- moved J5 6.13 mm to (58.0, 66.3)
- moved kibuzzard-69783B26 6.00 mm to (120.0, 138.5)
- moved J8 3.03 mm to (77.5, 97.2)
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Routing:
- net /Vehicle Control CAN-: track 81.9 -> 124.3 mm
- net /Vehicle Control CAN+: track 77.4 -> 115.2 mm
- net +BATT: track 188.2 -> 152.8 mm, vias 30 -> 23
- net /Arm Motor CAN-: track 51.3 -> 47.1 mm
- net /Arm Motor CAN+: track 45.2 -> 40.9 mm
- net GND: track 7.33 -> 10.4 mm, vias 64 -> 67
- net +12V: track 112.5 -> 111.2 mm, vias 5 -> 3
- net +5V: track 190.3 -> 191.1 mm, vias 3 -> 5
- net +3.3V: vias 3 -> 2

Commit message: Final Part 3
Parts:
- added C12: 63uF, Capacitor_SMD:CP_Elec_6.3x7.7, F.Cu at (60.8, 115.5)
- added C13: 63uF, Capacitor_SMD:CP_Elec_6.3x7.7, F.Cu at (59.0, 129.2)
- added C14: 63uF, Capacitor_SMD:CP_Elec_6.3x7.7, F.Cu at (50.9, 129.2)
- added C7: 63uF, Capacitor_SMD:CP_Elec_6.3x7.7, F.Cu at (60.8, 107.5)
- J12, J6: footprint Connector_AMASS:AMASS_XT60PW-F_1x02_P7.20mm_Horizontal -> Connector_AMASS:AMASS_XT60-F_1x02_P7.20mm_Vertical
- moved C1 17.2 mm to (66.3, 143.9), turned to -90 degrees
- moved JP1 15.6 mm to (64.0, 147.3), turned to 180 degrees
- moved R14 13.4 mm to (61.5, 148.2), turned to 90 degrees
- moved J6 11.6 mm to (58.5, 98.0), turned to 180 degrees
- moved kibuzzard-696EEFE3 10.4 mm to (47.0, 143.0), turned to 90 degrees
- moved R15 10.3 mm to (61.5, 141.0), turned to 90 degrees
- moved J11 7.87 mm to (56.2, 147.2), turned to 180 degrees
- moved J3 5.42 mm to (56.2, 138.8), turned to 180 degrees
- moved J12 4.69 mm to (58.6, 88.5), turned to 180 degrees
- moved J7 1.58 mm to (58.2, 77.3)
Routing:
- net /Vehicle Control CAN+: track 115.2 -> 131.5 mm
- net /Vehicle Control CAN-: track 124.3 -> 123.7 mm
- net +BATT: track 152.8 -> 152.6 mm, vias 23 -> 26
- net GND: vias 67 -> 68

Commit message: Details
Parts:
- moved C7 12.7 mm to (51.5, 116.2), turned to 180 degrees
- moved M2 6.05 mm to (70.0, 150.9), turned to 0 degrees
- moved G*** 5.53 mm to (75.6, 146.0)
- moved G*** 5.22 mm to (75.6, 149.8)
- moved C13 4.90 mm to (62.1, 125.4), turned to 0 degrees
- moved kibuzzard-6970222E 4.79 mm to (80.5, 159.0)
- moved D1 4.79 mm to (88.5, 156.5)
- moved D5 4.79 mm to (81.5, 151.5)
- moved D6 4.79 mm to (81.5, 156.5)
- moved D7 4.79 mm to (88.5, 151.6)
- moved R12 4.79 mm to (79.2, 156.5)
- moved R13 4.79 mm to (86.2, 156.5)
- moved R19 4.79 mm to (79.2, 151.6)
- moved R20 4.79 mm to (86.3, 151.6)
- moved kibuzzard-696EF04A 4.79 mm to (87.1, 159.0)
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Routing:
- net +BATT: track 152.6 -> 164.7 mm, vias 26 -> 20
- net +12V: track 111.2 -> 108.1 mm
- net +3.3V: track 157.9 -> 155.3 mm
- net +5V: track 190.8 -> 188.2 mm

Commit message: Review Changes
Parts:
- C10, C3, C8, C9: moved to B.Cu
- kibuzzard-69B0C619: moved to F.Cu
- moved G*** 65.6 mm to (12.5, 128.2)
- moved G*** 65.6 mm to (12.5, 132.0)
- moved H2 10.2 mm to (133.2, 155.8)
- moved J4 9.57 mm to (123.2, 156.4)
- moved kibuzzard-69B0C619 9.57 mm to (118.6, 153.9)
- moved D1 4.10 mm to (92.5, 156.4)
- moved D5 4.10 mm to (85.6, 151.4)
- moved D6 4.10 mm to (85.6, 156.4)
- moved D7 4.10 mm to (92.6, 151.5)
- moved R19 4.10 mm to (83.3, 151.4)
- moved R20 4.10 mm to (90.3, 151.5)
- moved kibuzzard-696EF04A 4.10 mm to (91.2, 158.9)
- moved R12 4.10 mm to (83.3, 156.4)
- moved R13 4.10 mm to (90.3, 156.4)
- moved kibuzzard-696EF05A 4.10 mm to (84.5, 153.9)
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Routing:
- net +5V: track 188.2 -> 183.1 mm
- net +BATT: track 164.7 -> 169.7 mm, vias 20 -> 22
- net +3.3V: track 155.3 -> 151.2 mm
- net /ESP0 3.3V: track 70.8 -> 74.9 mm
- net +12V: track 108.1 -> 109.6 mm
- net /Arm Motor CAN+: track 40.9 -> 39.8 mm
- net /Arm Motor CAN-: track 47.1 -> 46.2 mm
- net GND: vias 68 -> 75

Commit message: Odering Version
Parts:
- moved J6 2.10 mm to (58.2, 100.0)
- moved H2 0.89 mm to (134.0, 156.2)
Connections:
- J14 pad 4: /MOSI_ESP0 -> /ENCOD_MOSI
- J14 pad 5: /MISO_ESP0 -> /ENCOD_MISO
- J14 pad 6: /CLK_ESP0 -> /ENCOD_CLK
- J2 pad 5: /MOSI_ESP0 -> /ENCOD_MOSI
- J2 pad 6: /MISO_ESP0 -> /ENCOD_MISO
- J2 pad 7: /CLK_ESP0 -> /ENCOD_CLK
- U5 pad 28: unconnected-(U5-GPIO47-Pad28) -> /ENCOD_CLK
- U5 pad 29: /CLK_ESP0 -> /SPI_CLK
- U5 pad 30: /MISO_ESP0 -> /SPI_MISO
- U5 pad 31: unconnected-(U5-GPIO0-Pad31) -> /ENCOD_MISO
- U5 pad 33: /MOSI_ESP0 -> /SPI_MOSI
- U5 pad 35: /CS_Encoder_1 -> /ENCOD_MOSI
- U5 pad 41: unconnected-(U5-GPIO1/ADC1_CH0-Pad41) -> /CS_Encoder_1
- U9 pad 22: /CLK_ESP0 -> /SPI_CLK
- U9 pad 23: /MISO_ESP0 -> /SPI_MISO
- U9 pad 24: /MOSI_ESP0 -> /SPI_MOSI
Routing:
- net /CLK_ESP0: track 129.3 -> 0.00 mm
- net /MISO_ESP0: track 114.7 -> 0.00 mm
- net /ENCOD_CLK: track 0.00 -> 109.5 mm
- net /MOSI_ESP0: track 106.9 -> 0.00 mm
- net /ENCOD_MISO: track 0.00 -> 90.2 mm
- net /ENCOD_MOSI: track 0.00 -> 74.5 mm
- net /SPI_MOSI: track 0.00 -> 27.7 mm
- net /SPI_CLK: track 0.00 -> 23.9 mm
- net /SPI_MISO: track 0.00 -> 23.4 mm
- net /CS_Encoder_1: track 59.3 -> 42.6 mm
- net +BATT: track 169.7 -> 169.4 mm, vias 22 -> 18
- net GND: vias 75 -> 77
Other:
- outline, holes or cut-outs redrawn
- board text removed: "SPARKMAX XT60"

Commit message: silk
Parts:
- removed kibuzzard-696EEF69: G***, kibuzzard-696EEF69
- added kibuzzard-69CF1CE3: G***, kibuzzard-69CF1CE3, F.Cu at (71.6, 97.2)
- added kibuzzard-69CF1F55: G***, kibuzzard-69CF1F55, F.Cu at (68.0, 144.2)
- moved G*** 112.6 mm to (124.1, 147.5), turned to 90 degrees
- moved G*** 94.7 mm to (106.4, 140.6), turned to 90 degrees
- moved J4 71.3 mm to (83.4, 97.2), turned to -90 degrees
- moved M1 64.9 mm to (123.0, 151.1), turned to 0 degrees
- moved kibuzzard-696EEF9E 7.95 mm to (71.6, 105.2)
- moved J8 7.77 mm to (78.1, 105.0)
- moved kibuzzard-69B0C619 0.87 mm to (117.8, 154.2)
- moved C9 0.85 mm to (116.8, 114.5)
Routing:
- net +12V: track 109.6 -> 146.4 mm, vias 3 -> 1
- net +5V: track 183.1 -> 169.4 mm
- net /ESP0 3.3V: track 74.9 -> 75.7 mm
- net /Vehicle Control CAN-: track 123.7 -> 124.2 mm
- net GND: vias 77 -> 795
- net +BATT: vias 18 -> 21

Commit message: fixes for rev 2
Parts:
- removed U9: MCP251863T-E-9PX, Package_SO:SSOP-28_5.3x10.2mm_P0.65mm
- removed Y3: 40Mhz Crystal, Crystal:Crystal_SMD_3225-4Pin_3.2x2.5mm
- added JP2: SolderJumper_3_Open, Jumper:SolderJumper-3_P1.3mm_Open_RoundedPad1.0x1.5mm, B.Cu at (111.0, 122.9)
- added U6: MCP251863T-H-SS, Package_SO:SSOP-28_5.3x10.2mm_P0.65mm, B.Cu at (117.6, 122.4)
- added Y1: Crystal_GND24, Crystal:Crystal_SMD_3225-4Pin_3.2x2.5mm_HandSoldering, B.Cu at (128.6, 124.9)
- C2: value C_Small -> 4.7uF
- R8: value 2.21K ohm -> 2.00K ohm
- R9: value 3.32K ohm -> 3.01K ohm
- moved M1 10.0 mm to (133.0, 150.4)
- moved H2 10.0 mm to (124.0, 156.0)
- moved C8 9.33 mm to (114.0, 129.7)
- moved G*** 9.09 mm to (133.1, 146.3)
- moved G*** 6.05 mm to (101.4, 144.0)
- moved C4 5.23 mm to (129.6, 128.0)
- moved C6 3.29 mm to (127.9, 121.2)
- moved C10 1.20 mm to (120.0, 130.0)
- moved H1 0.20 mm to (50.0, 156.0)
- moved C2 0.17 mm to (105.5, 131.5)
Connections:
- U5 pad 17: unconnected-(U5-GPIO11/ADC2_CH0-Pad17) -> /CAN_STBY
Routing:
- net Net-(U6-RXCAN): track 0.00 -> 13.2 mm, vias 0 -> 2
- net Net-(U9-RXCAN): track 9.70 -> 0.00 mm, vias 2 -> 0
- net Net-(U6-TXCAN): track 0.00 -> 8.85 mm, vias 0 -> 2
- net Net-(U6-OSC1): track 7.12 -> 15.0 mm
- net +12V: track 146.4 -> 153.8 mm
- net Net-(U9-TXCAN): track 5.89 -> 0.00 mm
- net /ESP0 3.3V: track 75.7 -> 70.1 mm
- net +3.3V: track 151.2 -> 147.6 mm
- net Net-(JP2-C): track 0.00 -> 3.46 mm
- net /CAN_STBY: track 0.00 -> 3.25 mm
- net /ENCOD_CLK: track 109.5 -> 106.6 mm
- net GND: track 10.4 -> 7.94 mm, vias 795 -> 78
- net Net-(U6-OSC2): track 6.60 -> 8.45 mm
- net /Arm Motor CAN-: track 46.2 -> 47.5 mm
- net /Arm Motor CAN+: track 39.8 -> 40.9 mm
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- added copper zone on In1.Cu, net GND
- added copper zone on In2.Cu, net GND
Other:
- copper layers 2 -> 4
- board text added: "REV 2"

Commit message: More Changes for REV 2
Parts:
- H1, H2, H3, H4: footprint MountingHole:MountingHole_3.2mm_M3 -> MountingHole:MountingHole_3.2mm_M3_DIN965_Pad_TopBottom
- moved C5 1.27 mm to (112.0, 102.1)
- moved C6 0.20 mm to (127.9, 121.0)
Connections:
- U5 pad 31: /ENCOD_MISO -> unconnected-(U5-GPIO0-Pad31)
- U5 pad 40: unconnected-(U5-GPIO2/ADC1_CH1-Pad40) -> /ENCOD_MISO
Routing:
- net /ENCOD_MISO: track 90.2 -> 32.9 mm
- net /Vehicle Control CAN+: track 131.5 -> 103.3 mm
- net /Vehicle Control CAN-: track 124.2 -> 96.7 mm
- net +12V: track 153.8 -> 131.2 mm, vias 1 -> 2
- net +3.3V: track 147.6 -> 134.4 mm, vias 2 -> 3
- net /ESP0 3.3V: track 70.1 -> 65.6 mm
- net /Arm Motor CAN+: track 40.9 -> 38.9 mm
- net /CS_Encoder_2: track 27.9 -> 29.3 mm
- net /SPI_MOSI: track 27.7 -> 26.8 mm
- net +BATT: vias 19 -> 20
- net GND: vias 78 -> 81
- net +5V: vias 4 -> 6
- added copper zone on In1.Cu, net +12V
- removed copper zone on F.Cu, net +12V
- removed copper zone on F.Cu, net +5V
