File: Arm/Arm.kicad_sch (KiCad schematic)
At the start: 61 parts, among them J10 SparkMAX XT60 F, J11 CAN OUT, J12 SparkMAX XT60 F, J13 SparkMAX XT60 F, J14 Encoder 0, J2 Encoder Bundle, J3 CAN IN, J4 5V Swtich Power, J5 Power IN XT60 M, J6 SparkMAX XT60 F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

Commit message: Odering Version
Connections:
- net CS_Encoder_1: now also U5.41 (GPIO1/ADC1_CH0); no longer U5.35 (GPIO38)
- net SPI_CLK: now also U9.22 (SCK)
- net SPI_MISO: now also U9.23 (SDI)
- net SPI_MOSI: now also U9.24 (SDO)
- net ENCOD_CLK: now reaches U5.28 (GPIO47)
- net ENCOD_CLK: now also J14.6 (Pin_6), J2.7 (Pin_7)
- net ENCOD_MISO: now reaches U5.31 (GPIO0)
- net ENCOD_MISO: now also J14.5 (Pin_5), J2.6 (Pin_6)
- removed net CLK_ESP0: J14.6 (Pin_6), J2.7 (Pin_7), U9.22 (SCK)
- removed net MISO_ESP0: J14.5 (Pin_5), J2.6 (Pin_6), U9.23 (SDI)
- net MOSI_ESP0 renamed ENCOD_MOSI
- net ENCOD_MOSI: now also U5.35 (GPIO38)
Changed lines of the file:
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@@
 			"AAAAAAAAAAAAAAAAAAAAAAAAAAAAAAAAAAAAAAAAAAAAAAAAAAAAAAAAAAAAAAAAAAAAAAAAAAAA"
 			"AAAAAAAAAAAAAAAAAAAAAAAAAAAAAAAAAAAAAAAAAAAAAAAAAAAAAAAAAAAAAAAAAAAAAAAAAAAA"
+			"AAAAAAAAAAAAAAAAAAAAAAAAAAAAAAAAAAAAAAAAAAAAAAAAAAAAAAAAAAAAAAAAAAAAAAAAAAAA"
+			"AAAAAAAAAAAAAAAAAAAAAAAAAAAAAAAAAAAAAAAAAAAAAAAAAAAAAAAAAAAAAAAAAAAAAAAAAAAA"
+			"AAAAAAAAAAAAAAAAAAAAAAAAAAAAAAAAAAAAAAAAAAAAAAAAAAAAAAAAAAAAAAAAAAAAAAAAAAAA"
+			"AAAAAAAAAAAAAAAAAAAAAAAAAAAAAAAAAAAAAAAAAAAAAAAAAAAAAAAAAAAAAAAAAAAAAAAAAAAA"
+			"AAAAAAAAAAAAAAAAAAAAAAAAAAAAAAAAAAAAAAAAAAAAAAAAAAAAAAAAAAAAAAAAAAAAAAAAAAAA"
+			"AAAAAAAAAAAAAAAAAAAAAAAAAAAAAAAAAAAAAAAAAAAAAAAAAAAAAAAAAAAAAAAAAAAAAAAAAAAA"
+			"AAAAAAAAAAAAAAAAAAAAAAAAAAAAAAAAAAAAAAAAAAAAAAAAAAAAAAAAAAAAAAAAAAAAAAAAAAAA"
+			"AAAAAAAAAAAAAAAAAAAAAAAAAAAAAAAAAAAAAAAAAAAAAAAAAAAAAAAAAAAAAAAAAAAAAAAAAAAA"
+			"AAAAAAAAAAAAAAAAAAAAAAAAAAAAAAAAAAAAAAAAAAAAAAAAAAAAAAAAAAAAAAAAAAAAAAAAAAAA"
+			"AAAAAAAAAAAAAAAAAAAAAAAAAAAAAAAAAAAAAAAAAAAAAAAAAAAAAAAAAAAAAAAAAAAAAAAAAAAA"
+			"AAAAAAAAAAAAAAAAAAAAAAAAAAAAAAAAAAAAAAAAAAAAAAAAAAAAAAAAAAAAAAAAAAAAAAAAAAAA"
+			"AAAAAAAAAAAAAAAAAAAAAAAAAAAAAAAAAAAAAAAAAAAAAAAAAAAAAAAAAAAAAAAAAAAAAAAAAAAA"
+			"AAAAAAAAAAAAAAAAAAAAAAAAAAAAAAAAAAAAAAAAAAAAAAAAAAAAAAAAAAAAAAAAAAAAAAAAAAAA"
+			"AAAAAAAAAAAAAAAAAAAAAAAAAAAAAAAAAAAAAAAAAAAAAAAAAAAAAAAAAAAAAAAAAAAAAAAAAAAA"
+			"AAAAAAAAAAAAAAAAAAAAAAAAAAAAAAAAAAAAAAAAAAAAAAAAAAAAAAAAAAAAAAAAAAAAAAAAAAAA"
+			"AAAAAAAAAAAAAAAAAAAAAAAAAAAAAAAAAAAAAAAAAAAAAAAAAAAAAAAAAAAAAAAAAAAAAAAAAAAA"
+			"AAAAAAAAAAAAAAAAAAAAAAAAAAAAAAAAAAAAAAAAAAAAAAAAAAAAAAAAAAAAAAAAAAAAAAAAAAAA"
+			"AAAAAAAAAAAAAAAAAAAAAAAAAAAAAAAAAAAAAAAAAAAAAAAAAAAAAAAAAAAAAAAAAAAAAAAAAAAA"
 			"AAAAAAAAAAAAAAAAAAAAAAAAAAAAAAAAAAAAAAAAAAAAAAAAAAAAAAAAAA=="
 		)
@@
 			"AGUAAAB2AAAANQAAAHMAAAB6AAAAagAAAEIAAAB4AAAAdwAAAG0AAABQAAAAcgAAAFkAAABXAAAA"
 			"RAAAAHUAAABvAAAAUwAAAGwAAABGAAAAUAAAAHkAAABUAAAAYQAAAFAAAAA1AAAALwAAAHcAAABB"
-			"AAAAMAAAAHcAAABrAAAAYwAAAEwAAABqAAAAYQAAADIAAABHAAAAZwAAADcAAABxAA=="
+			"AAAAMAAAAHcAAABrAAAAYwAAAEwAAABqAAAAYQAAADIAAABHAAAAZwAAADcAAABxAAAARQAAAHAA"
+			"AABKAAAAZgAAAEoAAAB0AAAAQgAAAFIAAABSAAAAUgAAAFgAAABuAAAASAAAAEEAAABGAAAARgAA"
+			"AEYAAABGAAAAQQAAAEIAAABSAAAAUgAAAFIAAABRAAAAQQAAAFUAAABVAAAAVQAAAFUAAABBAAAA"
+			"RgAAAEYAAABGAAAARgAAAEEAAABCAAAAUgAAAFIAAABSAAAAUQAAAEEAAABVAAAAVQAAAFUAAABV"
+			"AAAAQQAAAEYAAABGAAAARgAAAEYAAABBAAAAQgAAAFIAAABSAAAAUgAAAFEAAABBAAAAVQAAAFUA"
+			"AABVAAAAVQAAAEEAAABGAAAARgAAAEYAAABGAAAAQQAAAEIAAABSAAAAUgAAAFIAAABRAAAAQQAA"
+			"AFUAAABVAAAAVQAAAFUAAABBAAAARgAAAEYAAABGAAAARgAAAEEAAABCAAAAUgAAAFIAAABSAAAA"
+			"UQAAAEEAAABVAAAAVQAAAFUAAABVAAAAQQAAAEYAAABGAAAARgAAAEYAAABBAAAASAAAAC8AAAAw"
+			"AAAAUAAAADMAAAA4AAAAbwAAAG8AAABvAAAAbwAAAEEAAABLAAAASwAAAEsAAABLAAAAQQAAAEMA"
+			"AABpAAAAaQAAAGkAAABnAAAAQQAAAG8AAABvAAAAbwAAAG8AAABBAAAASwAAAEsAAABLAAAASwAA"
+			"AEEAAABDAAAAaQAAAGkAAABpAAAAZwAAAEEAAABvAAAAbwAAAG8AAABvAAAAQQAAAEsAAABLAAAA"
+			"SwAAAEsAAABBAAAAQwAAAGkAAABpAAAAaQAAAGcAAABBAAAAbwAAAG8AAABvAAAAbwAAAEEAAABL"
+			"AAAASwAAAEsAAABLAAAAQQAAAEMAAABpAAAAaQAAAGkAAABnAAAAQQAAAG8AAABvAAAAbwAAAG8A"
+			"AABBAAAASwAAAEsAAABLAAAASwAAAEEAAABDAAAAaQAAAGkAAABpAAAAZwAAAEEAAABvAAAAbwAA"
+			"AG8AAABvAAAAQQAAAEsAAABLAAAASwAAAEsAAABBAAAAQwAAAGkAAABpAAAAaQAAAGcAAABBAAAA"
+			"bwAAAG8AAABvAAAAbwAAAEEAAABLAAAASwAAAEsAAABLAAAAQQAAAEMAAABpAAAAaQAAAGkAAABn"
+			"AAAAQQAAAHIAAAA4AAAAMQAAAHYAAABqAAAAegAAAC8AAAB3AAAAVAAAAG4AAAA4AAAATAAAAGYA"
+			"AABFAAAAMwAAAHgAAABkAAAAZQAAAGUAAABOAAAALwAAAEEAAABlAAAAdgAAAGYAAAA4AAAASQAA"
+			"AHQAAABlAAAANgAAAG4AAABLAAAAMQAAAHgAAABmAAAAVwAAAGMAAABsAAAAdAAAAA=="
 		)
 	)
@@
 		)
 	)
+	(label "SPI_MISO"
+		(at 255.27 53.34 180)
+		(effects
+			(font
+				(size 1.27 1.27)
+			)
+			(justify right bottom)
+		)
+	)
 	(label "Vehicle Control CAN+"
 		(at 226.06 177.8 0)
@@
 		)
 	)
+	(label "ENCOD_MISO"
+		(at 71.12 48.26 0)
+		(effects
+			(font
+				(size 1.27 1.27)
+			)
+			(justify left bottom)
+		)
+	)
 	(label "Arm Motor CAN-"
 		(at 200.66 175.26 0)
@@
 		)
 	)
+	(label "ENCOD_MISO"
+		(at 236.22 142.24 0)
+		(effects
+			(font
+				(size 1.27 1.27)
+			)
+			(justify left bottom)
+		)
+	)
 	(label "CS_Encoder_0"
 		(at 236.22 137.16 0)
@@
 		)
 	)
-	(label "MOSI_ESP0"
-		(at 236.22 139.7 0)
+	(label "Vehicle Control CAN-"
+		(at 170.18 175.26 0)
 		(effects
 			(font
@@
 		)
 	)
-	(label "Vehicle Control CAN-"
-		(at 170.18 175.26 0)
+	(label "ENCOD_MOSI"
+		(at 236.22 139.7 0)
 		(effects
 			(font
@@
 		)
 	)
-	(label "MOSI_ESP0"
-		(at 170.18 142.24 0)
-		(effects
-			(font
-				(size 1.27 1.27)
-			)
-			(justify left bottom)
-		)
-	)
 	(label "Arm Motor CAN-"
 		(at 288.29 57.15 0)
@@
 		)
 	)
-	(label "CS_Encoder_2"
-		(at 170.18 137.16 0)
+	(label "ENCOD_CLK"
+		(at 236.22 144.78 0)
 		(effects
 			(font
@@
 		)
 	)
-	(label "ESP0_TX-CAN_TX"
-		(at 186.69 63.5 0)
+	(label "CS_Encoder_2"
+		(at 170.18 137.16 0)
 		(effects
 			(font
@@
 		)
 	)
-	(label "CLK_ESP0"
-		(at 236.22 144.78 0)
+	(label "SPI_MOSI"
+		(at 255.27 55.88 180)
 		(effects
 			(font
 				(size 1.27 1.27)
 			)
-			(justify left bottom)
+			(justify right bottom)
 		)
 	)
-	(label "MISO_ESP0"
-		(at 236.22 142.24 0)
+	(label "ESP0_TX-CAN_TX"
+		(at 186.69 63.5 0)
 		(effects
 			(font
@@
 		)
 	)
-	(label "CS_Encoder_0"
-		(at 71.12 99.06 0)
+	(label "ENCOD_MOSI"
+		(at 71.12 101.6 0)
 		(effects
 			(font
@@
 		)
 	)
-	(label "CLK_ESP0"
-		(at 170.18 147.32 0)
+	(label "CS_Encoder_0"
+		(at 71.12 99.06 0)
 		(effects
 			(font
@@
 		)
 	)
-	(label "CLK_ESP0"
-		(at 255.27 60.96 180)
+	(label "ENCOD_CLK"
+		(at 71.12 109.22 0)
 		(effects
 			(font
 				(size 1.27 1.27)
 			)
-			(justify right bottom)
+			(justify left bottom)
 		)
 	)
@@
 		)
 	)
+	(label "ENCOD_MOSI"
+		(at 170.18 142.24 0)
+		(effects
+			(font
+				(size 1.27 1.27)
+			)
+			(justify left bottom)
+		)
+	)
+	(label "ENCOD_CLK"
+		(at 170.18 147.32 0)
+		(effects
+			(font
+				(size 1.27 1.27)
+			)
+			(justify left bottom)
+		)
+	)
 	(label "Vehicle Control CAN+"
 		(at 170.18 177.8 0)
@@
 		)
 	)
-	(label "CS_Encoder_1"
-		(at 71.12 101.6 0)
+	(label "ENCOD_MISO"
+		(at 170.18 144.78 0)
 		(effects
 			(font
@@
 		)
 	)
-	(label "MISO_ESP0"
-		(at 170.18 144.78 0)
+	(label "SPI_CLK"
+		(at 71.12 111.76 0)
 		(effects
 			(font
@@
 		)
 	)
-	(label "SPI_CLK"
-		(at 71.12 111.76 0)
+	(label "CS_Encoder_1"
+		(at 71.12 50.8 0)
 		(effects
 			(font
@@
 		)
 	)
-	(label "MISO_ESP0"
-		(at 255.27 53.34 180)
+	(label "SPI_CLK"
+		(at 255.27 60.96 180)
 		(effects
 			(font
