File: Arm/Arm.kicad_sch (KiCad schematic)
At the start: 61 parts, among them J10 SparkMAX XT60 F, J11 CAN OUT, J12 SparkMAX XT60 F, J13 SparkMAX XT60 F, J14 Encoder 0, J2 Encoder Bundle, J3 CAN IN, J4 5V Swtich Power, J5 Power IN XT60 M, J6 SparkMAX XT60 F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

Commit message: fixes for rev 2
Parts:
- removed U9: MCP251863T-E-9PX, Package_SO:SSOP-28_5.3x10.2mm_P0.65mm, symbol Interface_CAN_LIN:MCP251863T-E-9PX
- removed Y3: 40Mhz Crystal, Crystal:Crystal_SMD_3225-4Pin_3.2x2.5mm, symbol Device:Crystal_GND23
- added JP2: SolderJumper_3_Open, Jumper:SolderJumper-3_P1.3mm_Open_RoundedPad1.0x1.5mm, symbol Jumper:SolderJumper_3_Open
- added U6: MCP251863T-H-SS, Package_SO:SSOP-28_5.3x10.2mm_P0.65mm, symbol Interface_CAN_LIN:MCP251863T-H-SS
- added Y1: Crystal_GND24, Crystal:Crystal_SMD_3225-4Pin_3.2x2.5mm_HandSoldering, symbol Device:Crystal_GND24
- C2: value C_Small -> 4.7uF
- R8: value 2.21K ohm -> 2.00K ohm
- R9: value 3.32K ohm -> 3.01K ohm
Connections:
- net +5V: now also U6.25 (VCC)
- net Arm Motor CAN+: now also U6.4 (CANH)
- net Arm Motor CAN-: now also U6.3 (CANL)
- net CS_Motor_CAN: now also U6.13 (~{CS})
- net ESP0 3.3V: now also U6.1 (VIO), U6.14 (VDD)
- net GND: now also JP2.1 (A), U6.22 (VSS), U6.24 (GND), Y1.2, Y1.4
- net SPI_CLK: now also U6.9 (SCK)
- net SPI_MISO: now also U6.10 (SDI)
- net SPI_MOSI: now also U6.11 (SDO)
- net at C6.2: now also U6.20 (OSC2), Y1.1
- net at C4.2: now also U6.21 (OSC1), Y1.3
- net CAN_STBY: now reaches U5.17 (GPIO11/ADC2_CH0)
- net CAN_STBY: now also JP2.3 (B)
- new net: JP2.2 (C), U6.5 (STBY)
- new net: U6.15 (TXCAN), U6.23 (TXD)
- new net: U6.16 (RXCAN), U6.28 (RXD)
- no-connect marks 13 -> 12

Commit message: More Changes for REV 2
Parts:
- added JP3: SolderJumper_3_Open, Jumper:SolderJumper-3_P1.3mm_Open_RoundedPad1.0x1.5mm, symbol Jumper:SolderJumper_3_Open
- H1, H2, H3, H4: footprint MountingHole:MountingHole_3.2mm_M3 -> MountingHole:MountingHole_3.2mm_M3_DIN965_Pad_TopBottom
Connections:
- net ENCOD_MISO: now also U5.40 (GPIO2/ADC1_CH1); no longer U5.31 (GPIO0)
- net GND: now also JP3.1 (A)
- net at U5.3 (CHIP_PU): now also JP3.2 (C)
- new net +3V3: JP3.3 (B)
- no-connect marks 12 -> 11

Commit message: Final REV 2 Pt2
Connections:
- net +3V3 is gone; now on net +3.3V: JP3.3 (B)
- net CAN_STBY: now also U5.19 (GPIO13/ADC2_CH2); no longer U5.17 (GPIO11/ADC2_CH0)
- net MOTOR_CAN_INT1: now reaches U5.18 (GPIO12/ADC2_CH1)
- net MOTOR_CAN_INT1: now also U6.6 (~{INT1})
- net MOTOR_CAN_INT: now reaches U5.20 (GPIO14/ADC2_CH3)
- net MOTOR_CAN_INT: now also U6.19 (~{INT})
- net MOTOR_CAN_INT0: now reaches U6.7 (~{INT0})
- net MOTOR_CAN_INT0: now also U5.17 (GPIO11/ADC2_CH0)
- no-connect marks 11 -> 8
Other:
- moved on the sheet: C4, C6, Y1
